File: kicad/nowhere.kicad_pcb (KiCad board)
At the start: 2 copper layers, 24 parts, among them J1 DIN-4, J2 DIN-4, J3 DIN-4, J4 DIN-4, J5 DIN-4, J6 DIN-4, J7 DIN-4, J8 DIN-4, J9 Barrel_Jack, U1 Teensy3.6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

Commit message: Add PCB, gerber, and drill files
Parts:
- added REF**: MountingHole_2.5mm, MountingHole:MountingHole_2.5mm, F.Cu at (141.0, 80.0)
- added REF**: MountingHole_2.5mm, MountingHole:MountingHole_2.5mm, F.Cu at (141.0, 15.2)
- added REF**: MountingHole_2.5mm, MountingHole:MountingHole_2.5mm, F.Cu at (66.0, 15.2)
Routing:
- net +12V: track 0.00 -> 25.8 mm
- net Net-(D1-Pad1): track 21.4 -> 25.5 mm
Other:
- board outline added: 80 x 69.8 mm
Changed lines of the file:
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@@
   (general
     (thickness 1.6)
-    (drawings 1)
-    (tracks 183)
+    (drawings 7)
+    (tracks 191)
     (zones 0)
-    (modules 24)
+    (modules 27)
     (nets 113)
   )
@@
     (visible_elements FFFFFF7F)
     (pcbplotparams
-      (layerselection 0x010fc_ffffffff)
+      (layerselection 0x010f0_ffffffff)
       (usegerberextensions false)
       (usegerberattributes false)
@@
       (padsonsilk false)
       (subtractmaskfromsilk false)
-      (outputformat 4)
+      (outputformat 1)
       (mirror false)
       (drillshape 0)
       (scaleselection 1)
-      (outputdirectory ""))
+      (outputdirectory "gerber/"))
   )
   (net 0 "")
@@
     (uvia_drill 0.1)
     (add_net +5V)
+  )
+  (module MountingHole:MountingHole_2.5mm (layer F.Cu)
+    (at 140.97 80.01)
+    (descr "Mounting Hole 2.5mm, no annular")
+    (tags "mounting hole 2.5mm no annular")
+    (attr virtual)
+    (fp_text reference REF** (at 0 -3.5) (layer F.SilkS)
+      (effects (font (size 1 1) (thickness 0.15)))
+    )
+    (fp_text value MountingHole_2.5mm (at 0 3.5) (layer F.Fab)
+      (effects (font (size 1 1) (thickness 0.15)))
+    )
+    (fp_circle (center 0 0) (end 2.75 0) (layer F.CrtYd) (width 0.05))
+    (fp_circle (center 0 0) (end 2.5 0) (layer Cmts.User) (width 0.15))
+    (fp_text user %R (at 0.3 0) (layer F.Fab)
+      (effects (font (size 1 1) (thickness 0.15)))
+    )
+    (pad 1 np_thru_hole circle (at 0 0) (size 2.5 2.5) (drill 2.5) (layers *.Cu *.Mask))
+  )
+  (module MountingHole:MountingHole_2.5mm (layer F.Cu)
+    (at 140.97 15.24)
+    (descr "Mounting Hole 2.5mm, no annular")
+    (tags "mounting hole 2.5mm no annular")
+    (attr virtual)
+    (fp_text reference REF** (at 0 -3.5) (layer F.SilkS)
+      (effects (font (size 1 1) (thickness 0.15)))
+    )
+    (fp_text value MountingHole_2.5mm (at 0 3.5) (layer F.Fab)
+      (effects (font (size 1 1) (thickness 0.15)))
+    )
+    (fp_circle (center 0 0) (end 2.75 0) (layer F.CrtYd) (width 0.05))
+    (fp_circle (center 0 0) (end 2.5 0) (layer Cmts.User) (width 0.15))
+    (fp_text user %R (at 0.3 0) (layer F.Fab)
+      (effects (font (size 1 1) (thickness 0.15)))
+    )
+    (pad 1 np_thru_hole circle (at 0 0) (size 2.5 2.5) (drill 2.5) (layers *.Cu *.Mask))
+  )
+  (module MountingHole:MountingHole_2.5mm (layer F.Cu)
+    (at 66.04 15.24)
+    (descr "Mounting Hole 2.5mm, no annular")
+    (tags "mounting hole 2.5mm no annular")
+    (attr virtual)
+    (fp_text reference REF** (at 0 -3.5) (layer F.SilkS)
+      (effects (font (size 1 1) (thickness 0.15)))
+    )
+    (fp_text value MountingHole_2.5mm (at 0 3.5) (layer F.Fab)
+      (effects (font (size 1 1) (thickness 0.15)))
+    )
+    (fp_circle (center 0 0) (end 2.75 0) (layer F.CrtYd) (width 0.05))
+    (fp_circle (center 0 0) (end 2.5 0) (layer Cmts.User) (width 0.15))
+    (fp_text user %R (at 0.3 0) (layer F.Fab)
+      (effects (font (size 1 1) (thickness 0.15)))
+    )
+    (pad 1 np_thru_hole circle (at 0 0) (size 2.5 2.5) (drill 2.5) (layers *.Cu *.Mask))
   )
   (module Resistor_THT:R_Axial_DIN0207_L6.3mm_D2.5mm_P10.16mm_Horizontal (layer F.Cu)
@@
     )
   )
+  (gr_line (start 143.51 81.28) (end 143.51 82.55) (layer Edge.Cuts) (width 0.05))
+  (gr_line (start 63.5 82.55) (end 143.51 82.55) (layer Edge.Cuts) (width 0.05))
+  (gr_line (start 143.51 12.7) (end 143.51 81.28) (layer Edge.Cuts) (width 0.05))
+  (gr_line (start 63.5 12.7) (end 143.51 12.7) (layer Edge.Cuts) (width 0.05))
+  (gr_line (start 63.5 13.97) (end 63.5 12.7) (layer Edge.Cuts) (width 0.05))
+  (gr_line (start 63.5 82.55) (end 63.5 13.97) (layer Edge.Cuts) (width 0.05))
   (gr_text "N            v1\no\nwHere\n\nPaul Kiernan\nAlexis Schwerin" (at 78.74 40.64) (layer F.SilkS)
     (effects (font (size 1.25 1.25) (thickness 0.25)) (justify left))
   )
+  (segment (start 74.19 64.77) (end 72.39 64.77) (width 1) (layer F.Cu) (net 1))
+  (segment (start 78.74 69.32) (end 74.19 64.77) (width 1) (layer F.Cu) (net 1))
+  (segment (start 78.74 76.2) (end 78.74 69.32) (width 1) (layer F.Cu) (net 1))
+  (segment (start 72.39 64.77) (end 72.39 58.42) (width 1) (layer F.Cu) (net 1))
+  (segment (start 73.66 57.15) (end 73.66 54.61) (width 1) (layer F.Cu) (net 1))
+  (segment (start 72.39 58.42) (end 73.66 57.15) (width 1) (layer F.Cu) (net 1))
   (segment (start 82.827259 80.01) (end 85.09 80.01) (width 1) (layer B.Cu) (net 2))
   (segment (start 78.55 80.01) (end 82.827259 80.01) (width 1) (layer B.Cu) (net 2))
@@
   (segment (start 71.12 16.51) (end 69.569999 18.060001) (width 0.5) (layer F.Cu) (net 3))
   (segment (start 81.557259 57.15) (end 83.82 57.15) (width 0.5) (layer F.Cu) (net 4))
-  (segment (start 73.852498 57.15) (end 81.557259 57.15) (width 0.5) (layer F.Cu) (net 4))
-  (segment (start 71.96 55.257502) (end 73.852498 57.15) (width 0.5) (layer F.Cu) (net 4))
   (segment (start 71.96 54.61) (end 71.96 55.257502) (width 0.5) (layer F.Cu) (net 4))
   (segment (start 85.09 58.42) (end 83.82 57.15) (width 0.5) (layer F.Cu) (net 4))
   (segment (start 85.09 64.77) (end 85.09 58.42) (width 0.5) (layer F.Cu) (net 4))
+  (segment (start 71.96 53.962498) (end 71.96 54.61) (width 0.5) (layer F.Cu) (net 4))
+  (segment (start 72.662499 53.259999) (end 71.96 53.962498) (width 0.5) (layer F.Cu) (net 4))
+  (segment (start 79.929999 53.259999) (end 72.662499 53.259999) (width 0.5) (layer F.Cu) (net 4))
+  (segment (start 83.82 57.15) (end 79.929999 53.259999) (width 0.5) (layer F.Cu) (net 4))
   (segment (start 105.41 45.72) (end 114.3 36.83) (width 0.25) (layer F.Cu) (net 5))
   (segment (start 104.14 45.72) (end 105.41 45.72) (width 0.25) (layer F.Cu) (net 5))

Commit message: PCB version 2
Parts:
- added G***: LOGO, nowhere:the-man-silkscreen, F.Cu at (129.5, 80.0)
- added G***: LOGO, nowhere:nowhere-silkscreen-small, F.Cu at (87.6, 39.4)
- added G***: LOGO, nowhere:nowhere-silkscreen, B.Cu at (120.7, 38.1)
- added G***: LOGO, nowhere:nowhere-silkscreen, B.Cu at (96.5, 49.5)
- added G***: LOGO, nowhere:nowhere-silkscreen, B.Cu at (114.3, 69.8)
- added G***: LOGO, nowhere:nowhere-silkscreen, B.Cu at (82.5, 63.5)
- added G***: LOGO, nowhere:nowhere-silkscreen, B.Cu at (87.6, 33.0)
- added REF**: MountingHole_2.5mm, MountingHole:MountingHole_2.5mm, F.Cu at (137.2, 85.1)
- J1, J2, J3, J4, J5, J6, J7, J8: footprint Connector_Molex:Molex_Nano-Fit_105310-xx04_2x02_P2.50mm_Vertical -> Connector_Molex:Molex_Nano-Fit_105314-xx04_2x02_P2.50mm_Horizontal
- moved REF** 75.1 mm to (66.0, 85.1)
- moved J1 13.3 mm to (125.7, 40.6), turned to 0 degrees
- moved J2 13.0 mm to (125.7, 49.5), turned to 0 degrees
- moved J3 12.8 mm to (125.7, 58.4), turned to 0 degrees
- moved J4 12.7 mm to (125.7, 67.3), turned to 0 degrees
- moved J5 6.82 mm to (120.7, 73.7), turned to 270 degrees
- moved R8 5.68 mm to (119.4, 66.0)
- moved R1 5.68 mm to (119.4, 39.4)
- moved R2 5.68 mm to (119.4, 43.2)
- moved R3 5.68 mm to (119.4, 47.0)
- moved R4 5.68 mm to (119.4, 50.8)
- moved R5 5.68 mm to (119.4, 54.6)
- moved R6 5.68 mm to (119.4, 58.4)
- moved R7 5.68 mm to (119.4, 62.2)
- moved J6 5.66 mm to (111.8, 73.7), turned to 270 degrees
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Connections:
- J1 pad 1: +12V -> Net-(J1-Pad1)
- J2 pad 1: +12V -> Net-(J2-Pad1)
- J3 pad 1: +12V -> Net-(J3-Pad1)
- J4 pad 1: +12V -> Net-(J4-Pad1)
- J5 pad 1: +12V -> Net-(J5-Pad1)
- J6 pad 1: +12V -> Net-(J6-Pad1)
- J7 pad 1: +12V -> Net-(J7-Pad1)
- J8 pad 1: +12V -> Net-(J8-Pad1)
Routing:
- net GND: track 217.4 -> 0.00 mm
- net data4_out: track 29.4 -> 22.0 mm
- net data0_out: track 15.0 -> 7.91 mm
- net Net-(R6-Pad2): track 11.2 -> 5.08 mm
- net Net-(R3-Pad2): track 12.8 -> 6.66 mm
- net Net-(R2-Pad2): track 13.3 -> 7.18 mm
- net Net-(R5-Pad2): track 11.7 -> 5.61 mm
- net Net-(R4-Pad2): track 12.3 -> 6.13 mm
- net Net-(R1-Pad2): track 13.8 -> 8.45 mm
- net Net-(R7-Pad2): track 10.7 -> 5.61 mm
- net Net-(R8-Pad2): track 10.2 -> 6.13 mm
- net data1_out: track 15.6 -> 11.7 mm
- net data2_out: track 19.4 -> 16.6 mm
- net data3_out: track 23.8 -> 21.6 mm
- net Net-(D1-Pad1): track 25.5 -> 24.2 mm
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- added copper zone on B.Cu, net GND
Other:
- board size 80 x 69.8 mm -> 76.2 x 73.7 mm
- board text added: "Paul Kiernan Alexis Schwerin v2"
- board text removed: "N v1 o wHere Paul Kiernan Alexis Schwerin"
